Commit message: tryign to fix meshes not found error

File: src/kinova_arm/description/urdf/kinova_common.xacro (robot description, xacro)
@@ -17,9 +17,9 @@
     <xacro:macro name="kinova_armlink" params="link_name link_mesh ring_mesh:=ring_big use_ring_mesh:=false mesh_no">
         <link name="${link_name}">
-            <visual>
-                <geometry>
-                    <mesh
-                        filename="$(find kinova_arm)/description/meshes/${link_mesh}.dae"/>
-                </geometry>
+      <visual>
+        <geometry>
+          <mesh
+            filename="package://kinova_arm/description/meshes/${link_mesh}.STL"/>
+        </geometry>
                 <material name="carbon_fiber">
                     <color rgba="0.792156862745098 0.819607843137255 0.933333333333333 1" />
@@ -28,17 +28,17 @@
 	    <!-- Adding ring to the model -->
 	         <xacro:if value="${use_ring_mesh}">
-	           <visual>
-                <geometry>
-                    <mesh
-                        filename="$(find kinova_arm)/description/meshes/${ring_mesh}.dae"/>
-                </geometry>
-             </visual>
+         <visual>
+        <geometry>
+          <mesh
+            filename="package://kinova_arm/description/meshes/${ring_mesh}.STL"/>
+        </geometry>
+       </visual>
 	    </xacro:if>
-            <collision>
-                <geometry>
-                    <mesh
-                        filename="$(find kinova_arm)/description/meshes/${link_mesh}.dae"/>
-                </geometry>
-            </collision>
+      <collision>
+        <geometry>
+          <mesh
+            filename="package://kinova_arm/description/meshes/${link_mesh}.STL"/>
+        </geometry>
+      </collision>
 						<xacro:kinova_inertial mesh_no="${mesh_no}"/>
       </link>
