Commit message: fixed mesh loading error + fixed 2 finger hand

File: src/kinova_arm/description/urdf/j2n6s300.xacro (robot description, xacro)
@@ -24,5 +24,5 @@
     <xacro:property name="link_4_mesh" value="wrist" />
     <xacro:property name="link_5_mesh" value="wrist" />
-    <xacro:property name="link_6_mesh" value="hand_2finger" />
+    <xacro:property name="link_6_mesh" value="hand_3finger" />
     <!--Used for conditional arguments for setting inertial parameters
         base 0, shoulder 1, arm 2, forearm 3, wrist 4, arm_mico 5,
@@ -37,5 +37,5 @@
     <xacro:property name="link_4_mesh_no" value="4" />
     <xacro:property name="link_5_mesh_no" value="4" />
-    <xacro:property name="link_6_mesh_no" value="56" />
+    <xacro:property name="link_6_mesh_no" value="55" />
     <xacro:property name="joint_base" value="joint_base" />
     <xacro:property name="joint_base_type" value="fixed" />
@@ -114,5 +114,5 @@
         <xacro:kinova_virtual_link link_name="${prefix}_end_effector"/>
         <xacro:kinova_virtual_joint joint_name="${prefix}_joint_end_effector" type="${joint_end_effector_type}" parent="${prefix}_link_6" child="${prefix}_end_effector" joint_axis_xyz="${joint_end_effector_axis_xyz}" joint_origin_xyz="${joint_end_effector_origin_xyz}" joint_origin_rpy="${joint_end_effector_origin_rpy}" joint_lower_limit="0" joint_upper_limit="0"/>
-        <xacro:kinova_2fingers link_hand="${prefix}_link_6" prefix="${prefix}_"/>
+        <xacro:kinova_3fingers link_hand="${prefix}_link_6" prefix="${prefix}_"/>
     </xacro:macro>
 </root>

File: src/kinova_arm/description/urdf/kinova_common.xacro (robot description, xacro)
@@ -20,5 +20,5 @@
         <geometry>
           <mesh
-            filename="package://kinova_arm/description/meshes/${link_mesh}.STL"/>
+            filename="file://$(find kinova_arm)/description/meshes/${link_mesh}.STL"/>
         </geometry>
                 <material name="carbon_fiber">
@@ -31,5 +31,5 @@
         <geometry>
           <mesh
-            filename="package://kinova_arm/description/meshes/${ring_mesh}.STL"/>
+            filename="file://$(find kinova_arm)/description/meshes/${ring_mesh}.STL"/>
         </geometry>
        </visual>
@@ -38,5 +38,5 @@
         <geometry>
           <mesh
-            filename="package://kinova_arm/description/meshes/${link_mesh}.STL"/>
+            filename="file://$(find kinova_arm)/description/meshes/${link_mesh}.STL"/>
         </geometry>
       </collision>

File: src/kinova_arm/description/urdf/kinova_finger_set.xacro (robot description, xacro)
@@ -23,9 +23,3 @@
         <xacro:kinova_finger prefix="${prefix}" finger_number="3" hand="${link_hand}" finger_origin_xyz="-0.02226 -0.02707 -0.11482" finger_origin_rpy="-1.570796327 .649262481663582 -1.75545216211587"/>
     </xacro:macro>
-    <xacro:macro name="kinova_2fingers" params="link_hand prefix">
-        <!-- finger1 Rot := Ry((1/2)*Pi) . Rx(Pi) . Rz(-52.8*((1/180)*Pi)) -->
-        <xacro:kinova_finger prefix="${prefix}" finger_number="1" hand="${link_hand}" finger_origin_xyz="-0.0025 0.03095 -0.11482" finger_origin_rpy="-1.570796327 .649262481663582 1.57079632679490"/>
-        <!-- finger2 Rot := Ry((1/2)*Pi) . Rz(-52.8*((1/180)*Pi))  -->
-        <xacro:kinova_finger prefix="${prefix}" finger_number="2" hand="${link_hand}" finger_origin_xyz="-0.0025 -0.03095 -0.11482" finger_origin_rpy="-1.570796327 .649262481663582 -1.57079632679490"/>
-    </xacro:macro>
 </root>
