Commit message: new cmakelists.txt

File: kinova_moveit/config/moveit/j2n6s300.ros2_control.xacro (robot description, xacro)
@@ -1,96 +1,75 @@
 <?xml version="1.0"?>
 <robot xmlns:xacro="http://www.ros.org/wiki/xacro">
-    <xacro:macro name="j2n6s300_ros2_control" params="name initial_positions_file">
-        <xacro:property name="initial_positions" value="${xacro.load_yaml(initial_positions_file)['initial_positions']}"/>
-        <ros2_control name="${name}" type="system">
-            <hardware>
-                <!-- By default, set up controllers for simulation. This won't work on real hardware -->
-                <plugin>mock_components/GenericSystem</plugin>
-            </hardware>
-            <joint name="j2n6s300_joint_1">
-                <command_interface name="position"/>
-                <state_interface name="position">
-                  <param name="initial_value">${initial_positions['j2n6s300_joint_1']}</param>
-                </state_interface>
-                <state_interface name="velocity"/>
-            </joint>
-            <joint name="j2n6s300_joint_2">
-                <command_interface name="position"/>
-                <state_interface name="position">
-                  <param name="initial_value">${initial_positions['j2n6s300_joint_2']}</param>
-                </state_interface>
-                <state_interface name="velocity"/>
-            </joint>
-            <joint name="j2n6s300_joint_3">
-                <command_interface name="position"/>
-                <state_interface name="position">
-                  <param name="initial_value">${initial_positions['j2n6s300_joint_3']}</param>
-                </state_interface>
-                <state_interface name="velocity"/>
-            </joint>
-            <joint name="j2n6s300_joint_4">
-                <command_interface name="position"/>
-                <state_interface name="position">
-                  <param name="initial_value">${initial_positions['j2n6s300_joint_4']}</param>
-                </state_interface>
-                <state_interface name="velocity"/>
-            </joint>
-            <joint name="j2n6s300_joint_5">
-                <command_interface name="position"/>
-                <state_interface name="position">
-                  <param name="initial_value">${initial_positions['j2n6s300_joint_5']}</param>
-                </state_interface>
-                <state_interface name="velocity"/>
-            </joint>
-            <joint name="j2n6s300_joint_6">
-                <command_interface name="position"/>
-                <state_interface name="position">
-                  <param name="initial_value">${initial_positions['j2n6s300_joint_6']}</param>
-                </state_interface>
-                <state_interface name="velocity"/>
-            </joint>
-            <joint name="j2n6s300_joint_finger_1">
-                <command_interface name="position"/>
-                <state_interface name="position">
-                  <param name="initial_value">${initial_positions['j2n6s300_joint_finger_1']}</param>
-                </state_interface>
-                <state_interface name="velocity"/>
-            </joint>
-            <joint name="j2n6s300_joint_finger_tip_1">
-                <command_interface name="position"/>
-                <state_interface name="position">
-                  <param name="initial_value">${initial_positions['j2n6s300_joint_finger_tip_1']}</param>
-                </state_interface>
-                <state_interface name="velocity"/>
-            </joint>
-            <joint name="j2n6s300_joint_finger_2">
-                <command_interface name="position"/>
-                <state_interface name="position">
-                  <param name="initial_value">${initial_positions['j2n6s300_joint_finger_2']}</param>
-                </state_interface>
-                <state_interface name="velocity"/>
-            </joint>
-            <joint name="j2n6s300_joint_finger_tip_2">
-                <command_interface name="position"/>
-                <state_interface name="position">
-                  <param name="initial_value">${initial_positions['j2n6s300_joint_finger_tip_2']}</param>
-                </state_interface>
-                <state_interface name="velocity"/>
-            </joint>
-            <joint name="j2n6s300_joint_finger_3">
-                <command_interface name="position"/>
-                <state_interface name="position">
-                  <param name="initial_value">${initial_positions['j2n6s300_joint_finger_3']}</param>
-                </state_interface>
-                <state_interface name="velocity"/>
-            </joint>
-            <joint name="j2n6s300_joint_finger_tip_3">
-                <command_interface name="position"/>
-                <state_interface name="position">
-                  <param name="initial_value">${initial_positions['j2n6s300_joint_finger_tip_3']}</param>
-                </state_interface>
-                <state_interface name="velocity"/>
-            </joint>
-        </ros2_control>
+  <xacro:macro name="j2n6s300_ros2_control" params="name initial_positions_file">
+      <xacro:property name="initial_positions" value="${xacro.load_yaml(initial_positions_file)['initial_positions']}"/>
+    <xacro:macro name="connect_joint" params="prefix">
+      <joint name="j2n6s300_joint_${prefix}">
+        <command_interface name="velocity"/>
+        <state_interface name="position"/>
+        <state_interface name="velocity"/>
+        <state_interface name="current"/>
+        <state_interface name="voltage"/>
+      </joint>
     </xacro:macro>
+    <ros2_control name="{name}" type="system"/>
+      <hardware>
+        <!-- By default, set up controllers for simulation. This won't work on real hardware -->
+        <plugin>kinova_driver/KinovaSystemHardware</plugin>
+      </hardware>
+      <xacro:connect_joint prefix="1"/>
+      <xacro:connect_joint prefix="2"/>
+      <xacro:connect_joint prefix="3"/>
+      <xacro:connect_joint prefix="4"/>
+      <xacro:connect_joint prefix="5"/>
+      <xacro:connect_joint prefix="6"/>
+    </ros2_control>
+    <ros2_control name="${name}" type="system">
+      <hardware>
+          <!-- By default, set up controllers for simulation. This won't work on real hardware -->
+          <plugin>mock_components/GenericSystem</plugin>
+      </hardware>
+      <joint name="j2n6s300_joint_finger_1">
+          <command_interface name="position"/>
+          <state_interface name="position">
+            <param name="initial_value">${initial_positions['j2n6s300_joint_finger_1']}</param>
+          </state_interface>
+          <state_interface name="velocity"/>
+      </joint>
+      <joint name="j2n6s300_joint_finger_tip_1">
+          <command_interface name="position"/>
+          <state_interface name="position">
+            <param name="initial_value">${initial_positions['j2n6s300_joint_finger_tip_1']}</param>
+          </state_interface>
+          <state_interface name="velocity"/>
+      </joint>
+      <joint name="j2n6s300_joint_finger_2">
+          <command_interface name="position"/>
+          <state_interface name="position">
+            <param name="initial_value">${initial_positions['j2n6s300_joint_finger_2']}</param>
+          </state_interface>
+          <state_interface name="velocity"/>
+      </joint>
+      <joint name="j2n6s300_joint_finger_tip_2">
+          <command_interface name="position"/>
+          <state_interface name="position">
+            <param name="initial_value">${initial_positions['j2n6s300_joint_finger_tip_2']}</param>
+          </state_interface>
+          <state_interface name="velocity"/>
+      </joint>
+      <joint name="j2n6s300_joint_finger_3">
+          <command_interface name="position"/>
+          <state_interface name="position">
+            <param name="initial_value">${initial_positions['j2n6s300_joint_finger_3']}</param>
+          </state_interface>
+          <state_interface name="velocity"/>
+      </joint>
+      <joint name="j2n6s300_joint_finger_tip_3">
+          <command_interface name="position"/>
+          <state_interface name="position">
+            <param name="initial_value">${initial_positions['j2n6s300_joint_finger_tip_3']}</param>
+          </state_interface>
+          <state_interface name="velocity"/>
+      </joint>
+    </ros2_control>
+  </xacro:macro>
 </robot>
