Commit message: residual files from space_sinter

File: config/moveit/j2n6s300.urdf.xacro (robot description, xacro)
@@ -1,9 +1,9 @@
 <?xml version="1.0"?>
 <robot xmlns:xacro="http://www.ros.org/wiki/xacro" name="j2n6s300">
-    <xacro:arg name="initial_positions_file" default="$(find kinova_gen2)/config/initial_positions.yaml" />
+    <xacro:arg name="initial_positions_file" default="$(find space_sinter)/config/initial_positions.yaml" />
     <!-- Import j2n6s300 urdf file -->
-    <xacro:include filename="$(find kinova_gen2)/description/urdf/j2n6s300_standalone.xacro" />
+    <xacro:include filename="$(find space_sinter)/description/urdf/j2n6s300_standalone.xacro" />
     <!-- Import control_xacro -->
-    <xacro:include filename="$(find kinova_gen2)/config/moveit/j2n6s300.ros2_control.xacro" />
+    <xacro:include filename="$(find space_sinter)/config/moveit/j2n6s300.ros2_control.xacro" />
     <xacro:j2n6s300_ros2_control name="FakeSystem" initial_positions_file="$(arg initial_positions_file)"/>
 </robot>

File: description/urdf/j2n6s300.xacro (robot description, xacro)
@@ -14,8 +14,8 @@
     xmlns:physics="http://playerstage.sourceforge.net/gazebo/xmlschema/#physics"
     xmlns:xacro="http://www.ros.org/wiki/xacro">
-    <xacro:include filename="$(find kinova_gen2)/description/urdf/kinova_common.xacro" />
-    <xacro:include filename="$(find kinova_gen2)/description/urdf/kinova_finger_set.xacro" />
+    <xacro:include filename="$(find space_sinter)/description/urdf/kinova_common.xacro" />
+    <xacro:include filename="$(find space_sinter)/description/urdf/kinova_finger_set.xacro" />
     <!-- Import all Gazebo-customization elements -->
-    <xacro:include filename="$(find kinova_gen2)/description/urdf/kinova_gazebo.xacro" />
+    <xacro:include filename="$(find space_sinter)/description/urdf/kinova_gazebo.xacro" />
     <xacro:property name="link_base_mesh" value="base" />
     <xacro:property name="link_1_mesh" value="shoulder" />
@@ -98,18 +98,18 @@
     <xacro:macro name="j2n6s300" params="base_parent prefix:=j2n6s300">
     <xacro:gazebo_config robot_namespace="${prefix}"/>
-        <xacro:kinova_gen2link link_name="${prefix}_link_base" link_mesh="${link_base_mesh}" mesh_no="${link_base_mesh_no}"/>
-        <xacro:kinova_gen2joint joint_name="${prefix}_joint_base" type="${joint_base_type}" parent="${base_parent}" child="${prefix}_link_base" joint_axis_xyz="${joint_base_axis_xyz}" joint_origin_xyz="${joint_base_origin_xyz}" joint_origin_rpy="${joint_base_origin_rpy}" fixed="true"/>
-        <xacro:kinova_gen2link link_name="${prefix}_link_1" link_mesh="${link_1_mesh}" use_ring_mesh="true" mesh_no="${link_1_mesh_no}"/>
-        <xacro:kinova_gen2joint joint_name="${prefix}_joint_1" type="${joint_1_type}" parent="${prefix}_link_base" child="${prefix}_link_1" joint_axis_xyz="${joint_1_axis_xyz}" joint_origin_xyz="${joint_1_origin_xyz}" joint_origin_rpy="${joint_1_origin_rpy}" joint_velocity_limit="${joint_1_velocity_limit}" joint_torque_limit="${joint_1_torque_limit}"/>
-        <xacro:kinova_gen2link link_name="${prefix}_link_2" link_mesh="${link_2_mesh}" use_ring_mesh="true" mesh_no="${link_2_mesh_no}"/>
-        <xacro:kinova_gen2joint joint_name="${prefix}_joint_2" type="${joint_2_type}" parent="${prefix}_link_1" child="${prefix}_link_2" joint_axis_xyz="${joint_2_axis_xyz}" joint_origin_xyz="${joint_2_origin_xyz}" joint_origin_rpy="${joint_2_origin_rpy}" joint_lower_limit="${joint_2_lower_limit}" joint_upper_limit="${joint_2_upper_limit}" joint_velocity_limit="${joint_2_velocity_limit}" joint_torque_limit="${joint_2_torque_limit}"/>
-        <xacro:kinova_gen2link link_name="${prefix}_link_3" link_mesh="${link_3_mesh}" use_ring_mesh="true" mesh_no="${link_3_mesh_no}"/>
-        <xacro:kinova_gen2joint joint_name="${prefix}_joint_3" type="${joint_3_type}" parent="${prefix}_link_2" child="${prefix}_link_3" joint_axis_xyz="${joint_3_axis_xyz}" joint_origin_xyz="${joint_3_origin_xyz}" joint_origin_rpy="${joint_3_origin_rpy}" joint_lower_limit="${joint_3_lower_limit}" joint_upper_limit="${joint_3_upper_limit}" joint_velocity_limit="${joint_3_velocity_limit}" joint_torque_limit="${joint_3_torque_limit}"/>
-        <xacro:kinova_gen2link link_name="${prefix}_link_4" link_mesh="${link_4_mesh}" use_ring_mesh="true" ring_mesh="ring_small" mesh_no="${link_4_mesh_no}"/>
-        <xacro:kinova_gen2joint joint_name="${prefix}_joint_4" type="${joint_4_type}" parent="${prefix}_link_3" child="${prefix}_link_4" joint_axis_xyz="${joint_4_axis_xyz}" joint_origin_xyz="${joint_4_origin_xyz}" joint_origin_rpy="${joint_4_origin_rpy}" joint_velocity_limit="${joint_4_velocity_limit}" joint_torque_limit="${joint_4_torque_limit}"/>
-        <xacro:kinova_gen2link link_name="${prefix}_link_5" link_mesh="${link_5_mesh}" use_ring_mesh="true" ring_mesh="ring_small" mesh_no="${link_5_mesh_no}"/>
-        <xacro:kinova_gen2joint joint_name="${prefix}_joint_5" type="${joint_5_type}" parent="${prefix}_link_4" child="${prefix}_link_5" joint_axis_xyz="${joint_5_axis_xyz}" joint_origin_xyz="${joint_5_origin_xyz}" joint_origin_rpy="${joint_5_origin_rpy}" joint_velocity_limit="${joint_5_velocity_limit}" joint_torque_limit="${joint_5_torque_limit}"/>
-        <xacro:kinova_gen2link link_name="${prefix}_link_6" link_mesh="${link_6_mesh}" use_ring_mesh="true" ring_mesh="ring_small" mesh_no="${link_6_mesh_no}"/>
-        <xacro:kinova_gen2joint joint_name="${prefix}_joint_6" type="${joint_6_type}" parent="${prefix}_link_5" child="${prefix}_link_6" joint_axis_xyz="${joint_6_axis_xyz}" joint_origin_xyz="${joint_6_origin_xyz}" joint_origin_rpy="${joint_6_origin_rpy}" joint_velocity_limit="${joint_6_velocity_limit}" joint_torque_limit="${joint_6_torque_limit}"/>
+        <xacro:space_sinterlink link_name="${prefix}_link_base" link_mesh="${link_base_mesh}" mesh_no="${link_base_mesh_no}"/>
+        <xacro:space_sinterjoint joint_name="${prefix}_joint_base" type="${joint_base_type}" parent="${base_parent}" child="${prefix}_link_base" joint_axis_xyz="${joint_base_axis_xyz}" joint_origin_xyz="${joint_base_origin_xyz}" joint_origin_rpy="${joint_base_origin_rpy}" fixed="true"/>
+        <xacro:space_sinterlink link_name="${prefix}_link_1" link_mesh="${link_1_mesh}" use_ring_mesh="true" mesh_no="${link_1_mesh_no}"/>
+        <xacro:space_sinterjoint joint_name="${prefix}_joint_1" type="${joint_1_type}" parent="${prefix}_link_base" child="${prefix}_link_1" joint_axis_xyz="${joint_1_axis_xyz}" joint_origin_xyz="${joint_1_origin_xyz}" joint_origin_rpy="${joint_1_origin_rpy}" joint_velocity_limit="${joint_1_velocity_limit}" joint_torque_limit="${joint_1_torque_limit}"/>
+        <xacro:space_sinterlink link_name="${prefix}_link_2" link_mesh="${link_2_mesh}" use_ring_mesh="true" mesh_no="${link_2_mesh_no}"/>
+        <xacro:space_sinterjoint joint_name="${prefix}_joint_2" type="${joint_2_type}" parent="${prefix}_link_1" child="${prefix}_link_2" joint_axis_xyz="${joint_2_axis_xyz}" joint_origin_xyz="${joint_2_origin_xyz}" joint_origin_rpy="${joint_2_origin_rpy}" joint_lower_limit="${joint_2_lower_limit}" joint_upper_limit="${joint_2_upper_limit}" joint_velocity_limit="${joint_2_velocity_limit}" joint_torque_limit="${joint_2_torque_limit}"/>
+        <xacro:space_sinterlink link_name="${prefix}_link_3" link_mesh="${link_3_mesh}" use_ring_mesh="true" mesh_no="${link_3_mesh_no}"/>
+        <xacro:space_sinterjoint joint_name="${prefix}_joint_3" type="${joint_3_type}" parent="${prefix}_link_2" child="${prefix}_link_3" joint_axis_xyz="${joint_3_axis_xyz}" joint_origin_xyz="${joint_3_origin_xyz}" joint_origin_rpy="${joint_3_origin_rpy}" joint_lower_limit="${joint_3_lower_limit}" joint_upper_limit="${joint_3_upper_limit}" joint_velocity_limit="${joint_3_velocity_limit}" joint_torque_limit="${joint_3_torque_limit}"/>
+        <xacro:space_sinterlink link_name="${prefix}_link_4" link_mesh="${link_4_mesh}" use_ring_mesh="true" ring_mesh="ring_small" mesh_no="${link_4_mesh_no}"/>
+        <xacro:space_sinterjoint joint_name="${prefix}_joint_4" type="${joint_4_type}" parent="${prefix}_link_3" child="${prefix}_link_4" joint_axis_xyz="${joint_4_axis_xyz}" joint_origin_xyz="${joint_4_origin_xyz}" joint_origin_rpy="${joint_4_origin_rpy}" joint_velocity_limit="${joint_4_velocity_limit}" joint_torque_limit="${joint_4_torque_limit}"/>
+        <xacro:space_sinterlink link_name="${prefix}_link_5" link_mesh="${link_5_mesh}" use_ring_mesh="true" ring_mesh="ring_small" mesh_no="${link_5_mesh_no}"/>
+        <xacro:space_sinterjoint joint_name="${prefix}_joint_5" type="${joint_5_type}" parent="${prefix}_link_4" child="${prefix}_link_5" joint_axis_xyz="${joint_5_axis_xyz}" joint_origin_xyz="${joint_5_origin_xyz}" joint_origin_rpy="${joint_5_origin_rpy}" joint_velocity_limit="${joint_5_velocity_limit}" joint_torque_limit="${joint_5_torque_limit}"/>
+        <xacro:space_sinterlink link_name="${prefix}_link_6" link_mesh="${link_6_mesh}" use_ring_mesh="true" ring_mesh="ring_small" mesh_no="${link_6_mesh_no}"/>
+        <xacro:space_sinterjoint joint_name="${prefix}_joint_6" type="${joint_6_type}" parent="${prefix}_link_5" child="${prefix}_link_6" joint_axis_xyz="${joint_6_axis_xyz}" joint_origin_xyz="${joint_6_origin_xyz}" joint_origin_rpy="${joint_6_origin_rpy}" joint_velocity_limit="${joint_6_velocity_limit}" joint_torque_limit="${joint_6_torque_limit}"/>
         <xacro:kinova_virtual_link link_name="${prefix}_end_effector"/>
         <xacro:kinova_virtual_joint joint_name="${prefix}_joint_end_effector" type="${joint_end_effector_type}" parent="${prefix}_link_6" child="${prefix}_end_effector" joint_axis_xyz="${joint_end_effector_axis_xyz}" joint_origin_xyz="${joint_end_effector_origin_xyz}" joint_origin_rpy="${joint_end_effector_origin_rpy}" joint_lower_limit="0" joint_upper_limit="0"/>

File: description/urdf/j2n6s300_standalone.xacro (robot description, xacro)
@@ -14,5 +14,5 @@
     xmlns:physics="http://playerstage.sourceforge.net/gazebo/xmlschema/#physics"
 	xmlns:xacro="http://www.ros.org/wiki/xacro" name="j2n6s300">
-  <xacro:include filename="$(find kinova_gen2)/description/urdf/j2n6s300.xacro"/>
+  <xacro:include filename="$(find space_sinter)/description/urdf/j2n6s300.xacro"/>
   <link name="root"/>
   <!-- for gazebo -->

File: description/urdf/kinova_common.xacro (robot description, xacro)
@@ -13,12 +13,12 @@
     xmlns:physics="http://playerstage.sourceforge.net/gazebo/xmlschema/#physics"
 	xmlns:xacro="http://www.ros.org/wiki/xacro">
-<xacro:include filename="$(find kinova_gen2)/description/urdf/kinova_inertial.xacro" />
+<xacro:include filename="$(find space_sinter)/description/urdf/kinova_inertial.xacro" />
     <xacro:property name="J_PI" value="3.1415926535897931" />
-    <xacro:macro name="kinova_gen2link" params="link_name link_mesh ring_mesh:=ring_big use_ring_mesh:=false mesh_no">
+    <xacro:macro name="space_sinterlink" params="link_name link_mesh ring_mesh:=ring_big use_ring_mesh:=false mesh_no">
         <link name="${link_name}">
       <visual>
         <geometry>
           <mesh
-            filename="file://$(find kinova_gen2)/description/meshes/${link_mesh}.STL"/>
+            filename="file://$(find space_sinter)/description/meshes/${link_mesh}.STL"/>
         </geometry>
                 <material name="carbon_fiber">
@@ -31,5 +31,5 @@
         <geometry>
           <mesh
-            filename="file://$(find kinova_gen2)/description/meshes/${ring_mesh}.STL"/>
+            filename="file://$(find space_sinter)/description/meshes/${ring_mesh}.STL"/>
         </geometry>
        </visual>
@@ -38,5 +38,5 @@
         <geometry>
           <mesh
-            filename="file://$(find kinova_gen2)/description/meshes/${link_mesh}.STL"/>
+            filename="file://$(find space_sinter)/description/meshes/${link_mesh}.STL"/>
         </geometry>
       </collision>
@@ -53,5 +53,5 @@
   -->
   <xacro:property name="dummy_default_value" value="1234567890"/>
-  <xacro:macro name="kinova_gen2joint" params="joint_name
+  <xacro:macro name="space_sinterjoint" params="joint_name
                                               type
                                               parent
@@ -126,5 +126,5 @@
     </xacro:macro>
     <xacro:macro name="kinova_finger" params="prefix finger_number hand finger_origin_xyz finger_origin_rpy">
-        <xacro:kinova_gen2link link_name="${prefix}link_finger_${finger_number}" link_mesh="finger_proximal" mesh_no="57"/>
+        <xacro:space_sinterlink link_name="${prefix}link_finger_${finger_number}" link_mesh="finger_proximal" mesh_no="57"/>
         <joint name="${prefix}joint_finger_${finger_number}" type="revolute">
             <parent link="${hand}"/>
@@ -144,5 +144,5 @@
 					</actuator>
 		    </transmission>
-        <xacro:kinova_gen2link link_name="${prefix}link_finger_tip_${finger_number}" link_mesh="finger_distal" mesh_no="58"/>
+        <xacro:space_sinterlink link_name="${prefix}link_finger_tip_${finger_number}" link_mesh="finger_distal" mesh_no="58"/>
         <joint name="${prefix}joint_finger_tip_${finger_number}" type="revolute">
             <parent link="${prefix}link_finger_${finger_number}"/>

File: description/urdf/kinova_finger_set.xacro (robot description, xacro)
@@ -14,5 +14,5 @@
     xmlns:physics="http://playerstage.sourceforge.net/gazebo/xmlschema/#physics"
     xmlns:xacro="http://www.ros.org/wiki/xacro">
-    <xacro:include filename="$(find kinova_gen2)/description/urdf/kinova_common.xacro" />
+    <xacro:include filename="$(find space_sinter)/description/urdf/kinova_common.xacro" />
     <xacro:macro name="kinova_3fingers" params="link_hand prefix">
         <!-- finger1 Rot := Ry(96.12*((1/180)*Pi)) . Rx(1.2*((1/180)*Pi)) . Rz(52.52*((1/180)*Pi)) -->
