Commit message: fixed sim behavior, should work properly now

File: space_sinter/config/moveit/j2n6s300.ros2_control_fake.xacro (robot description, xacro)
@@ -8,6 +8,6 @@
                 <plugin>mock_components/GenericSystem</plugin>
             </hardware>
-            <joint name="j2n6s300_joint_1">
-                <<command_interface name="velocity"/>/>
+      <joint name="j2n6s300_joint_1">
+        <command_interface name="position"/>
                 <state_interface name="position">
                   <param name="initial_value">${initial_positions['j2n6s300_joint_1']}</param>
@@ -15,6 +15,6 @@
                 <state_interface name="velocity"/>
             </joint>
-            <joint name="j2n6s300_joint_2">
-                <<command_interface name="velocity"/>/>
+      <joint name="j2n6s300_joint_2">
+        <command_interface name="position"/>
                 <state_interface name="position">
                   <param name="initial_value">${initial_positions['j2n6s300_joint_2']}</param>
@@ -22,6 +22,6 @@
                 <state_interface name="velocity"/>
             </joint>
-            <joint name="j2n6s300_joint_3">
-                <<command_interface name="velocity"/>/>
+      <joint name="j2n6s300_joint_3">
+        <command_interface name="position"/>
                 <state_interface name="position">
                   <param name="initial_value">${initial_positions['j2n6s300_joint_3']}</param>
@@ -29,6 +29,6 @@
                 <state_interface name="velocity"/>
             </joint>
-            <joint name="j2n6s300_joint_4">
-                <<command_interface name="velocity"/>/>
+      <joint name="j2n6s300_joint_4">
+        <command_interface name="position"/>
                 <state_interface name="position">
                   <param name="initial_value">${initial_positions['j2n6s300_joint_4']}</param>
@@ -36,6 +36,6 @@
                 <state_interface name="velocity"/>
             </joint>
-            <joint name="j2n6s300_joint_5">
-                <<command_interface name="velocity"/>/>
+      <joint name="j2n6s300_joint_5">
+        <command_interface name="position"/>
                 <state_interface name="position">
                   <param name="initial_value">${initial_positions['j2n6s300_joint_5']}</param>
@@ -43,6 +43,6 @@
                 <state_interface name="velocity"/>
             </joint>
-            <joint name="j2n6s300_joint_6">
-                <<command_interface name="velocity"/>/>
+      <joint name="j2n6s300_joint_6">
+        <command_interface name="position"/>
                 <state_interface name="position">
                   <param name="initial_value">${initial_positions['j2n6s300_joint_6']}</param>
@@ -50,6 +50,6 @@
                 <state_interface name="velocity"/>
             </joint>
-            <joint name="j2n6s300_joint_finger_1">
-                <<command_interface name="velocity"/>/>
+      <joint name="j2n6s300_joint_finger_1">
+        <command_interface name="position"/>
                 <state_interface name="position">
                   <param name="initial_value">${initial_positions['j2n6s300_joint_finger_1']}</param>
@@ -57,6 +57,6 @@
                 <state_interface name="velocity"/>
             </joint>
-            <joint name="j2n6s300_joint_finger_tip_1">
-                <<command_interface name="velocity"/>/>
+      <joint name="j2n6s300_joint_finger_tip_1">
+        <command_interface name="position"/>
                 <state_interface name="position">
                   <param name="initial_value">${initial_positions['j2n6s300_joint_finger_tip_1']}</param>
@@ -64,6 +64,6 @@
                 <state_interface name="velocity"/>
             </joint>
-            <joint name="j2n6s300_joint_finger_2">
-                <<command_interface name="velocity"/>/>
+      <joint name="j2n6s300_joint_finger_2">
+        <command_interface name="position"/>
                 <state_interface name="position">
                   <param name="initial_value">${initial_positions['j2n6s300_joint_finger_2']}</param>
@@ -71,6 +71,6 @@
                 <state_interface name="velocity"/>
             </joint>
-            <joint name="j2n6s300_joint_finger_tip_2">
-                <<command_interface name="velocity"/>/>
+      <joint name="j2n6s300_joint_finger_tip_2">
+        <command_interface name="position"/>
                 <state_interface name="position">
                   <param name="initial_value">${initial_positions['j2n6s300_joint_finger_tip_2']}</param>
@@ -78,6 +78,6 @@
                 <state_interface name="velocity"/>
             </joint>
-            <joint name="j2n6s300_joint_finger_3">
-                <<command_interface name="velocity"/>/>
+      <joint name="j2n6s300_joint_finger_3">
+        <command_interface name="position"/>
                 <state_interface name="position">
                   <param name="initial_value">${initial_positions['j2n6s300_joint_finger_3']}</param>
@@ -85,6 +85,6 @@
                 <state_interface name="velocity"/>
             </joint>
-            <joint name="j2n6s300_joint_finger_tip_3">
-                <<command_interface name="velocity"/>/>
+      <joint name="j2n6s300_joint_finger_tip_3">
+        <command_interface name="position"/>
                 <state_interface name="position">
                   <param name="initial_value">${initial_positions['j2n6s300_joint_finger_tip_3']}</param>

Commit message: final changes for suntracking

File: space_sinter/config/moveit/j2n6s300.ros2_control_fake.xacro (robot description, xacro)
@@ -8,6 +8,6 @@
                 <plugin>mock_components/GenericSystem</plugin>
             </hardware>
-            <joint name="j2n6s300_joint_1">
-                <command_interface name="position"/>
+      <joint name="j2n6s300_joint_1">
+        <command_interface name="position"/>
                 <state_interface name="position">
                   <param name="initial_value">${initial_positions['j2n6s300_joint_1']}</param>
@@ -15,6 +15,6 @@
                 <state_interface name="velocity"/>
             </joint>
-            <joint name="j2n6s300_joint_2">
-                <command_interface name="position"/>
+      <joint name="j2n6s300_joint_2">
+        <command_interface name="position"/>
                 <state_interface name="position">
                   <param name="initial_value">${initial_positions['j2n6s300_joint_2']}</param>
@@ -22,6 +22,6 @@
                 <state_interface name="velocity"/>
             </joint>
-            <joint name="j2n6s300_joint_3">
-                <command_interface name="position"/>
+      <joint name="j2n6s300_joint_3">
+        <command_interface name="position"/>
                 <state_interface name="position">
                   <param name="initial_value">${initial_positions['j2n6s300_joint_3']}</param>
@@ -29,6 +29,6 @@
                 <state_interface name="velocity"/>
             </joint>
-            <joint name="j2n6s300_joint_4">
-                <command_interface name="position"/>
+      <joint name="j2n6s300_joint_4">
+        <command_interface name="position"/>
                 <state_interface name="position">
                   <param name="initial_value">${initial_positions['j2n6s300_joint_4']}</param>
@@ -36,6 +36,6 @@
                 <state_interface name="velocity"/>
             </joint>
-            <joint name="j2n6s300_joint_5">
-                <command_interface name="position"/>
+      <joint name="j2n6s300_joint_5">
+        <command_interface name="position"/>
                 <state_interface name="position">
                   <param name="initial_value">${initial_positions['j2n6s300_joint_5']}</param>
@@ -43,6 +43,6 @@
                 <state_interface name="velocity"/>
             </joint>
-            <joint name="j2n6s300_joint_6">
-                <command_interface name="position"/>
+      <joint name="j2n6s300_joint_6">
+        <command_interface name="position"/>
                 <state_interface name="position">
                   <param name="initial_value">${initial_positions['j2n6s300_joint_6']}</param>
@@ -50,6 +50,6 @@
                 <state_interface name="velocity"/>
             </joint>
-            <joint name="j2n6s300_joint_finger_1">
-                <command_interface name="position"/>
+      <joint name="j2n6s300_joint_finger_1">
+        <command_interface name="position"/>
                 <state_interface name="position">
                   <param name="initial_value">${initial_positions['j2n6s300_joint_finger_1']}</param>
@@ -57,6 +57,6 @@
                 <state_interface name="velocity"/>
             </joint>
-            <joint name="j2n6s300_joint_finger_tip_1">
-                <command_interface name="position"/>
+      <joint name="j2n6s300_joint_finger_tip_1">
+        <command_interface name="position"/>
                 <state_interface name="position">
                   <param name="initial_value">${initial_positions['j2n6s300_joint_finger_tip_1']}</param>
@@ -64,6 +64,6 @@
                 <state_interface name="velocity"/>
             </joint>
-            <joint name="j2n6s300_joint_finger_2">
-                <command_interface name="position"/>
+      <joint name="j2n6s300_joint_finger_2">
+        <command_interface name="position"/>
                 <state_interface name="position">
                   <param name="initial_value">${initial_positions['j2n6s300_joint_finger_2']}</param>
@@ -71,6 +71,6 @@
                 <state_interface name="velocity"/>
             </joint>
-            <joint name="j2n6s300_joint_finger_tip_2">
-                <command_interface name="position"/>
+      <joint name="j2n6s300_joint_finger_tip_2">
+        <command_interface name="position"/>
                 <state_interface name="position">
                   <param name="initial_value">${initial_positions['j2n6s300_joint_finger_tip_2']}</param>
@@ -78,6 +78,6 @@
                 <state_interface name="velocity"/>
             </joint>
-            <joint name="j2n6s300_joint_finger_3">
-                <command_interface name="position"/>
+      <joint name="j2n6s300_joint_finger_3">
+        <command_interface name="position"/>
                 <state_interface name="position">
                   <param name="initial_value">${initial_positions['j2n6s300_joint_finger_3']}</param>
@@ -85,6 +85,6 @@
                 <state_interface name="velocity"/>
             </joint>
-            <joint name="j2n6s300_joint_finger_tip_3">
-                <command_interface name="position"/>
+      <joint name="j2n6s300_joint_finger_tip_3">
+        <command_interface name="position"/>
                 <state_interface name="position">
                   <param name="initial_value">${initial_positions['j2n6s300_joint_finger_tip_3']}</param>
