Commit message: working mock configuration

File: src/sinter_arm_description/sinter_arm_description/urdf/j2n6s300_urdf_macro.xacro (robot description, xacro)
@@ -17,5 +17,5 @@
       <visual>
         <geometry>
-          <mesh filename="package://example_arm_description/meshes/visual/base.dae"/>
+          <mesh filename="package://sinter_arm_description/meshes/visual/base.dae"/>
         </geometry>
         <material name="carbon_fiber">
@@ -25,5 +25,5 @@
       <collision>
         <geometry>
-          <mesh filename="package://example_arm_description/meshes/collision/base.STL"/>
+          <mesh filename="package://sinter_arm_description/meshes/collision/base.STL"/>
         </geometry>
       </collision>
@@ -47,16 +47,16 @@
       <visual>
         <geometry>
-          <mesh filename="package://example_arm_description/meshes/visual/shoulder.dae"/>
-        </geometry>
-        <material name="carbon_fiber"/>
-      </visual>
-      <visual>
-        <geometry>
-          <mesh filename="package://example_arm_description/meshes/visual/ring_big.dae"/>
-        </geometry>
-      </visual>
-      <collision>
-        <geometry>
-          <mesh filename="package://example_arm_description/meshes/collision/shoulder.STL"/>
+          <mesh filename="package://sinter_arm_description/meshes/visual/shoulder.dae"/>
+        </geometry>
+        <material name="carbon_fiber"/>
+      </visual>
+      <visual>
+        <geometry>
+          <mesh filename="package://sinter_arm_description/meshes/visual/ring_big.dae"/>
+        </geometry>
+      </visual>
+      <collision>
+        <geometry>
+          <mesh filename="package://sinter_arm_description/meshes/collision/shoulder.STL"/>
         </geometry>
       </collision>
@@ -83,16 +83,16 @@
       <visual>
         <geometry>
-          <mesh filename="package://example_arm_description/meshes/visual/arm.dae"/>
-        </geometry>
-        <material name="carbon_fiber"/>
-      </visual>
-      <visual>
-        <geometry>
-          <mesh filename="package://example_arm_description/meshes/visual/ring_big.dae"/>
-        </geometry>
-      </visual>
-      <collision>
-        <geometry>
-          <mesh filename="package://example_arm_description/meshes/collision/arm.STL"/>
+          <mesh filename="package://sinter_arm_description/meshes/visual/arm.dae"/>
+        </geometry>
+        <material name="carbon_fiber"/>
+      </visual>
+      <visual>
+        <geometry>
+          <mesh filename="package://sinter_arm_description/meshes/visual/ring_big.dae"/>
+        </geometry>
+      </visual>
+      <collision>
+        <geometry>
+          <mesh filename="package://sinter_arm_description/meshes/collision/arm.STL"/>
         </geometry>
       </collision>
@@ -119,16 +119,16 @@
       <visual>
         <geometry>
-          <mesh filename="package://example_arm_description/meshes/visual/forearm.dae"/>
-        </geometry>
-        <material name="carbon_fiber"/>
-      </visual>
-      <visual>
-        <geometry>
-          <mesh filename="package://example_arm_description/meshes/visual/ring_big.dae"/>
-        </geometry>
-      </visual>
-      <collision>
-        <geometry>
-          <mesh filename="package://example_arm_description/meshes/collision/forearm.STL"/>
+          <mesh filename="package://sinter_arm_description/meshes/visual/forearm.dae"/>
+        </geometry>
+        <material name="carbon_fiber"/>
+      </visual>
+      <visual>
+        <geometry>
+          <mesh filename="package://sinter_arm_description/meshes/visual/ring_big.dae"/>
+        </geometry>
+      </visual>
+      <collision>
+        <geometry>
+          <mesh filename="package://sinter_arm_description/meshes/collision/forearm.STL"/>
         </geometry>
       </collision>
@@ -155,16 +155,16 @@
       <visual>
         <geometry>
-          <mesh filename="package://example_arm_description/meshes/visual/wrist.dae"/>
-        </geometry>
-        <material name="carbon_fiber"/>
-      </visual>
-      <visual>
-        <geometry>
-          <mesh filename="package://example_arm_description/meshes/visual/ring_small.dae"/>
-        </geometry>
-      </visual>
-      <collision>
-        <geometry>
-          <mesh filename="package://example_arm_description/meshes/collision/wrist.STL"/>
+          <mesh filename="package://sinter_arm_description/meshes/visual/wrist.dae"/>
+        </geometry>
+        <material name="carbon_fiber"/>
+      </visual>
+      <visual>
+        <geometry>
+          <mesh filename="package://sinter_arm_description/meshes/visual/ring_small.dae"/>
+        </geometry>
+      </visual>
+      <collision>
+        <geometry>
+          <mesh filename="package://sinter_arm_description/meshes/collision/wrist.STL"/>
         </geometry>
       </collision>
@@ -191,16 +191,16 @@
       <visual>
         <geometry>
-          <mesh filename="package://example_arm_description/meshes/visual/wrist.dae"/>
-        </geometry>
-        <material name="carbon_fiber"/>
-      </visual>
-      <visual>
-        <geometry>
-          <mesh filename="package://example_arm_description/meshes/visual/ring_small.dae"/>
-        </geometry>
-      </visual>
-      <collision>
-        <geometry>
-          <mesh filename="package://example_arm_description/meshes/collision/wrist.STL"/>
+          <mesh filename="package://sinter_arm_description/meshes/visual/wrist.dae"/>
+        </geometry>
+        <material name="carbon_fiber"/>
+      </visual>
+      <visual>
+        <geometry>
+          <mesh filename="package://sinter_arm_description/meshes/visual/ring_small.dae"/>
+        </geometry>
+      </visual>
+      <collision>
+        <geometry>
+          <mesh filename="package://sinter_arm_description/meshes/collision/wrist.STL"/>
         </geometry>
       </collision>
@@ -273,5 +273,15 @@
       <parent link="${prefix}_link_6"/>
       <child link="${prefix}_lens"/>
-      <origin xyz="0 0 -0.3" rpy="0 ${PI/2} 0"/>
+      <origin xyz="0 0 -0.3" rpy="${-PI/2} 0 ${-PI/2}"/>
+    </joint>
+    <!-- ========================================== -->
+    <!--   Focal Point (400mm along lens Z-axis)    -->
+    <!--   Virtual frame — no geometry/inertia      -->
+    <!-- ========================================== -->
+    <link name="${prefix}_focal_point"/>
+    <joint name="${prefix}_focal_point_joint" type="fixed">
+      <parent link="${prefix}_lens"/>
+      <child link="${prefix}_focal_point"/>
+      <origin xyz="0 0 0.4" rpy="0 0 0"/>
     </joint>
   </xacro:macro>

File: src/sinter_arm_drivers/ros2_control_interfaces/urdf/j2n6s300_physical_ros2_control_macro.xacro (robot description, xacro)
@@ -1,36 +1,43 @@
 <?xml version="1.0"?>
 <robot xmlns:xacro="http://wiki.ros.org/xacro">
-  <xacro:macro name="r6bot_control">
+  <xacro:macro name="j2n6s300_control">
     <ros2_control name="j2n6s300" type="system">
       <joint name="j2n6s300_joint_1">
-        <command_interface name="position"/>
+        <command_interface name="velocity"/>
         <state_interface name="position"/>
         <state_interface name="velocity"/>
+        <state_interface name="effort"/>
       </joint>
       <joint name="j2n6s300_joint_2">
-        <command_interface name="position"/>
+        <command_interface name="velocity"/>
         <state_interface name="position"/>
         <state_interface name="velocity"/>
+        <state_interface name="effort"/>
       </joint>
       <joint name="j2n6s300_joint_3">
-        <command_interface name="position"/>
+        <command_interface name="velocity"/>
         <state_interface name="position"/>
         <state_interface name="velocity"/>
+        <state_interface name="effort"/>
       </joint>
       <joint name="j2n6s300_joint_4">
-        <command_interface name="position"/>
+        <command_interface name="velocity"/>
         <state_interface name="position"/>
         <state_interface name="velocity"/>
+        <state_interface name="effort"/>
       </joint>
       <joint name="j2n6s300_joint_5">
-        <command_interface name="position"/>
+        <command_interface name="velocity"/>
         <state_interface name="position"/>
         <state_interface name="velocity"/>
+        <state_interface name="effort"/>
       </joint>
       <joint name="j2n6s300_joint_6">
-        <command_interface name="position"/>
+        <command_interface name="velocity"/>
         <state_interface name="position"/>
         <state_interface name="velocity"/>
+        <state_interface name="effort"/>
       </joint>
+    <!-- replace with some plugin for real hardware -->
       <hardware>
         <plugin>mock_components/GenericSystem</plugin>

File: src/sinter_robot_mock/urdf/j2n6s300.urdf.xacro (robot description, xacro)
@@ -13,3 +13,8 @@
   <link name="world"/>
   <xacro:j2n6s300_description base_parent="world"/>
+   <!-- Mock arm hardware -->
+  <xacro:if value="${'$(arg hardware_interface)' == 'mock'}">
+    <xacro:include filename="$(find ros2_control_interfaces)/urdf/j2n6s300_mock_ros2_control_macro.xacro"/>
+    <xacro:j2n6s300_control/>
+  </xacro:if>
 </robot>

Commit message: added camera optical frame

File: src/sinter_arm_description/sinter_arm_description/urdf/j2n6s300_urdf_macro.xacro (robot description, xacro)
@@ -248,7 +248,7 @@
     <link name="${prefix}_lens">
       <visual>
-        <origin xyz="0 0 0" rpy="0 0 0"/>
-        <geometry>
-          <box size="0.6 0.6 0.03"/>
+        <origin xyz="0 -0.01002 0.00827" rpy="0 0 0"/>
+        <geometry>
+          <box size="0.500 0.532 0.025"/>
         </geometry>
         <material name="lens_glass">
@@ -257,7 +257,7 @@
       </visual>
       <collision>
-        <origin xyz="0 0 0" rpy="0 0 0"/>
-        <geometry>
-          <box size="0.6 0.6 0.03"/>
+        <origin xyz="0 -0.27602 -0.00827" rpy="0 0 0"/>
+        <geometry>
+          <box size="0.500 0.532 0.025"/>
         </geometry>
       </collision>
@@ -273,5 +273,5 @@
       <parent link="${prefix}_link_6"/>
       <child link="${prefix}_lens"/>
-      <origin xyz="0 0 -0.3" rpy="${-PI/2} 0 ${-PI/2}"/>
+      <origin xyz="-0.00827 0 -0.27602" rpy="${-PI/2} 0 ${-PI/2}"/>
     </joint>
     <!-- ========================================== -->
@@ -285,4 +285,14 @@
       <origin xyz="0 0 0.4" rpy="0 0 0"/>
     </joint>
+    <!-- ========================================== -->
+    <!--   Camera Frame (reference middle of lens)  -->
+    <!--   Virtual frame — no geometry/inertia      -->
+    <!-- ========================================== -->
+    <link name="${prefix}_suncam_optical"/>
+    <joint name="${prefix}_suncam_joint" type="fixed">
+      <parent link="${prefix}_lens"/>
+      <child link="${prefix}_suncam_optical"/>
+      <origin xyz="-0.09436 -0.203 -0.03567" rpy="${PI} 0 0"/>
+    </joint>
   </xacro:macro>
 </robot>

Commit message: moving sort of

File: src/sinter_arm_description/sinter_arm_description/urdf/j2n6s300_urdf_macro.xacro (robot description, xacro)
@@ -257,5 +257,5 @@
       </visual>
       <collision>
-        <origin xyz="0 -0.27602 -0.00827" rpy="0 0 0"/>
+        <origin xyz="0 -0.01002 0.00827" rpy="0 0 0"/>
         <geometry>
           <box size="0.500 0.532 0.025"/>

File: src/sinter_arm_drivers/ros2_control_interfaces/urdf/j2n6s300_physical_ros2_control_macro.xacro (robot description, xacro)
@@ -4,5 +4,5 @@
     <ros2_control name="j2n6s300" type="system">
       <joint name="j2n6s300_joint_1">
-        <!-- <command_interface name="position"/> -->
+        <command_interface name="position"/>
         <command_interface name="velocity"/>
         <state_interface name="position"/>
@@ -11,5 +11,5 @@
       </joint>
       <joint name="j2n6s300_joint_2">
-        <!-- <command_interface name="position"/> -->
+        <command_interface name="position"/>
         <command_interface name="velocity"/>
         <state_interface name="position"/>
@@ -18,5 +18,5 @@
       </joint>
       <joint name="j2n6s300_joint_3">
-        <!-- <command_interface name="position"/> -->
+        <command_interface name="position"/>
         <command_interface name="velocity"/>
         <state_interface name="position"/>
@@ -25,5 +25,5 @@
       </joint>
       <joint name="j2n6s300_joint_4">
-        <!-- <command_interface name="position"/> -->
+        <command_interface name="position"/>
         <command_interface name="velocity"/>
         <state_interface name="position"/>
@@ -32,5 +32,5 @@
       </joint>
       <joint name="j2n6s300_joint_5">
-        <!-- <command_interface name="position"/> -->
+        <command_interface name="position"/>
         <command_interface name="velocity"/>
         <state_interface name="position"/>
@@ -39,5 +39,5 @@
       </joint>
       <joint name="j2n6s300_joint_6">
-        <!-- <command_interface name="position"/> -->
+        <command_interface name="position"/>
         <command_interface name="velocity"/>
         <state_interface name="position"/>

Commit message: changed urdf a lil

File: src/sinter_arm_description/sinter_arm_description/urdf/j2n6s300_urdf_macro.xacro (robot description, xacro)
@@ -293,5 +293,5 @@
       <parent link="${prefix}_lens"/>
       <child link="${prefix}_suncam_optical"/>
-      <origin xyz="-0.09436 -0.203 -0.03567" rpy="${PI} 0 0"/>
+      <origin xyz="-0.065 -0.203 -0.03567" rpy="${PI} 0 0"/>
     </joint>
   </xacro:macro>

Commit message: working movement driver, and added point cloud functionality

File: src/sinter_arm_description/sinter_arm_description/urdf/j2n6s300_urdf_macro.xacro (robot description, xacro)
@@ -293,5 +293,15 @@
       <parent link="${prefix}_lens"/>
       <child link="${prefix}_suncam_optical"/>
-      <origin xyz="-0.065 -0.203 -0.03567" rpy="${PI} 0 0"/>
+      <origin xyz="0.065 -0.203 -0.03567" rpy="${PI} 0 0"/>
+    </joint>
+    <!-- ========================================== -->
+    <!--   Realsense Camera Frame                   -->
+    <!--   Virtual frame — no geometry/inertia      -->
+    <!-- ========================================== -->
+    <link name="realsense_${prefix}"/>
+    <joint name="${prefix}_realsense_joint" type="fixed">
+      <parent link="${prefix}_lens"/>
+      <child link="realsense_${prefix}"/>
+      <origin xyz="-0.065 -0.203 -0.03567" rpy="${-PI/2} 0 ${PI}"/>
     </joint>
   </xacro:macro>

Commit message: semi working behavior, sun tracking behavior node is working appropriately

File: src/sinter_arm_description/sinter_arm_description/urdf/j2n6s300_urdf_macro.xacro (robot description, xacro)
@@ -283,5 +283,5 @@
       <parent link="${prefix}_lens"/>
       <child link="${prefix}_focal_point"/>
-      <origin xyz="0 0 0.4" rpy="0 0 0"/>
+      <origin xyz="0 0 0.4" rpy="${PI} 0 0"/>
     </joint>
     <!-- ========================================== -->

Commit message: added description changes

File: src/sinter_arm_description/sinter_arm_description/urdf/j2n6s300_urdf_macro.xacro (robot description, xacro)
@@ -273,5 +273,5 @@
       <parent link="${prefix}_link_6"/>
       <child link="${prefix}_lens"/>
-      <origin xyz="-0.00827 0 -0.27602" rpy="${-PI/2} 0 ${-PI/2}"/>
+      <origin xyz="-0.00827 0 -0.27602" rpy="${-PI/2} 0 0"/>
     </joint>
     <!-- ========================================== -->
@@ -293,5 +293,5 @@
       <parent link="${prefix}_lens"/>
       <child link="${prefix}_suncam_optical"/>
-      <origin xyz="0.065 -0.203 -0.03567" rpy="${PI} 0 0"/>
+      <origin xyz="0.065 -0.20452 -0.04178" rpy="${PI} 0 0"/>
     </joint>
     <!-- ========================================== -->
@@ -303,5 +303,5 @@
       <parent link="${prefix}_lens"/>
       <child link="realsense_${prefix}"/>
-      <origin xyz="-0.065 -0.203 -0.03567" rpy="${-PI/2} 0 ${PI}"/>
+      <origin xyz="-0.12645 -0.24618 -0.01158" rpy="${-PI/2} 0 ${PI}"/>
     </joint>
   </xacro:macro>
