Commit message: refactored sinter hardware driver

File: src/sinter_arm_description/sinter_arm_description/urdf/j2n6s300.urdf.xacro (robot description, xacro)
@@ -1,13 +1,14 @@
 <?xml version="1.0"?>
 <!--
-  Top-level Kinova Jaco2 j2n6s300 URDF (with lens, no gripper).
+  Top-level Kinova Jaco2 j2n6s300 URDF (with sinter end effector, no gripper).
   Xacro hierarchy:
     - package://sinter_arm_description/urdf/j2n6s300.urdf.xacro          (this file)
-      - package://sinter_arm_description/urdf/j2n6s300_urdf_macro.xacro  (arm + lens macro)
+      - package://sinter_arm_description/urdf/j2n6s300_urdf_macro.xacro  (arm macro)
+        - package://sinter_arm_description/urdf/end_effector_urdf_macro.xacro  (lens, sun cam, RealSense)
   Usage:
     xacro j2n6s300.urdf.xacro
 -->
 <robot xmlns:xacro="http://www.ros.org/wiki/xacro" name="j2n6s300">
-  <!-- Arm description macro (6 DOF + lens payload) -->
+  <!-- Arm description macro (6 DOF + end effector) -->
   <xacro:include filename="$(find sinter_arm_description)/urdf/j2n6s300_urdf_macro.xacro"/>
   <link name="world"/>

File: src/sinter_arm_description/sinter_arm_description/urdf/j2n6s300_urdf_macro.xacro (robot description, xacro)
@@ -1,7 +1,9 @@
 <?xml version="1.0"?>
 <robot xmlns:xacro="http://www.ros.org/wiki/xacro">
+  <xacro:include filename="$(find sinter_arm_description)/urdf/end_effector_urdf_macro.xacro"/>
   <!--
     Kinova Jaco2 6DOF Non-Spherical (j2n6s300)
-    6 DOF arm with 600x600x30mm lens payload (replaces gripper).
+    6 DOF arm with the sinter end effector (lens, sun camera, RealSense) replacing the gripper.
+    End effector is defined in end_effector_urdf_macro.xacro.
     Follows PickNik xacro naming conventions:
     - *_urdf_macro.xacro : macro definitions only, no output when included
@@ -224,5 +226,5 @@
     <!--    Link 6 - End Cap / Mount (continuous)   -->
     <!-- ========================================== -->
-    <!-- Link 6 is a virtual mount point: gripper/end effector removed, lens attaches here -->
+    <!-- Link 6 is a virtual mount point: gripper removed, end effector attaches here -->
     <link name="${prefix}_link_6">
       <inertial>
@@ -243,66 +245,8 @@
     </joint>
     <!-- ========================================== -->
-    <!--        Lens Payload (600x600x30mm)         -->
+    <!--   End Effector (lens, sun cam, RealSense)  -->
     <!--   Fixed to link_6, replaces gripper        -->
     <!-- ========================================== -->
-    <link name="${prefix}_lens">
-      <visual>
-        <origin xyz="0 -0.01002 0.00827" rpy="0 0 0"/>
-        <geometry>
-          <box size="0.500 0.532 0.025"/>
-        </geometry>
-        <material name="lens_glass">
-          <color rgba="0.3 0.3 0.8 0.5"/>
-        </material>
-      </visual>
-      <collision>
-        <origin xyz="0 -0.01002 0.00827" rpy="0 0 0"/>
-        <geometry>
-          <box size="0.500 0.532 0.025"/>
-        </geometry>
-      </collision>
-      <inertial>
-        <mass value="5.0"/>
-        <origin xyz="0 0 0"/>
-        <inertia ixx="0.150375" ixy="0" ixz="0"
-                 iyy="0.150375" iyz="0"
-                 izz="0.300000"/>
-      </inertial>
-    </link>
-    <joint name="${prefix}_lens_joint" type="fixed">
-      <parent link="${prefix}_link_6"/>
-      <child link="${prefix}_lens"/>
-      <origin xyz="-0.00827 0 -0.27602" rpy="${-PI/2} 0 0"/>
-    </joint>
-    <!-- ========================================== -->
-    <!--   Focal Point (400mm along lens Z-axis)    -->
-    <!--   Virtual frame — no geometry/inertia      -->
-    <!-- ========================================== -->
-    <link name="${prefix}_focal_point"/>
-    <joint name="${prefix}_focal_point_joint" type="fixed">
-      <parent link="${prefix}_lens"/>
-      <child link="${prefix}_focal_point"/>
-      <origin xyz="0 0 0.4" rpy="${PI} 0 0"/>
-    </joint>
-    <!-- ========================================== -->
-    <!--   Camera Frame (reference middle of lens)  -->
-    <!--   Virtual frame — no geometry/inertia      -->
-    <!-- ========================================== -->
-    <link name="${prefix}_suncam_optical"/>
-    <joint name="${prefix}_suncam_joint" type="fixed">
-      <parent link="${prefix}_lens"/>
-      <child link="${prefix}_suncam_optical"/>
-      <origin xyz="0.065 -0.20452 -0.04178" rpy="${PI} 0 0"/>
-    </joint>
-    <!-- ========================================== -->
-    <!--   Realsense Camera Frame                   -->
-    <!--   Virtual frame — no geometry/inertia      -->
-    <!-- ========================================== -->
-    <link name="realsense_${prefix}"/>
-    <joint name="${prefix}_realsense_joint" type="fixed">
-      <parent link="${prefix}_lens"/>
-      <child link="realsense_${prefix}"/>
-      <origin xyz="-0.12645 -0.24618 -0.01158" rpy="${-PI/2} 0 ${PI}"/>
-    </joint>
+    <xacro:sinter_end_effector parent="${prefix}_link_6"/>
   </xacro:macro>
 </robot>

File: src/sinter_arm_drivers/ros2_control_interfaces/urdf/j2n6s300_physical_ros2_control_macro.xacro (robot description, xacro)
@@ -47,6 +47,11 @@
       <hardware>
         <plugin>kinova_driver/KinovaSystemHardware</plugin>
-        <param name="state_following_offset">0.0</param>
-        <param name="calculate_dynamics">true</param>
+        <!-- Optional; defaults shown. See kinova_system_hardware.hpp. -->
+        <!-- <param name="serial_number"></param> -->
+        <param name="position_kp">5.0</param>
+        <param name="max_joint_velocity_deg">100.0</param>
+        <param name="io_rate_hz">100</param>
+        <param name="command_timeout_ms">100</param>
+        <param name="max_consecutive_io_errors">10</param>
       </hardware>
     </ros2_control>
