Commit message: last commit post showcase

File: src/sinter_robot_hw/urdf/j2n6s300.urdf.xacro (robot description, xacro)
@@ -12,4 +12,5 @@
   <xacro:include filename="$(find sinter_arm_description)/urdf/j2n6s300_urdf_macro.xacro"/>
   <link name="world"/>
+  <!-- <link name="world_rotated"/> -->
   <xacro:j2n6s300_description base_parent="world"/>
    <!-- Mock arm hardware -->

File: src/sinter_robot_mock/urdf/j2n6s300.urdf.xacro (robot description, xacro)
@@ -12,4 +12,5 @@
   <xacro:include filename="$(find sinter_arm_description)/urdf/j2n6s300_urdf_macro.xacro"/>
   <link name="world"/>
+  <!-- <link name="world_rotated"/> -->
   <xacro:j2n6s300_description base_parent="world"/>
    <!-- Mock arm hardware -->
